File: Multimeter.sch (KiCad schematic (older format))
At the start: 41 parts, among them J1 Conn_01x01, J2 Conn_01x01, J3 Conn_01x01, J4 Screw_Terminal_01x02, Q1 SQ3989EV, Q2 SQ3989EV, Q3 MMBT3906, Q4 MMBT3906, Q5 MMBT3906, Q6 MMBT3906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

Commit message: Fixed symbol mismatch
The pins for the TLV274 symbol were incorrect.
Parts:
- removed U1: TLV274CDR, Package_SO:SOIC-14_3.9x8.7mm_P1.27mm, symbol Amplifier_Operational:TLV9004xRUCR
- added U1: TLC274, Package_SO:SOIC-14_3.9x8.7mm_P1.27mm, symbol Amplifier_Operational:TLC274
- gave numbers to parts that had none: 1
Other:
- moved on the sheet: D3, D4, R8
Changed lines of the file:
@@
 	4900 4950 4900 5400
-$Comp
-L Amplifier_Operational:TLV9004xRUCR U1
-U 1 1 614A3ED4
-P 5700 4200
-F 0 "U1" H 5750 4400 50  0000 C CNN
-F 1 "TLV274CDR" H 5750 4500 50  0000 C CNN
-F 2 "Package_SO:SOIC-14_3.9x8.7mm_P1.27mm" H 5700 4200 50  0001 C CNN
-F 3 "https://www.ti.com/lit/ds/slos351e/slos351e.pdf" H 5750 4400 50  0001 C CNN
-	1    5700 4200
-	1    0    0    1
-$EndComp
-$Comp
-L Amplifier_Operational:TLV9004xRUCR U1
-U 5 1 614A5727
-P 6600 5400
-F 0 "U1" H 6558 5446 50  0000 L CNN
-F 1 "TLV274CDR" H 6558 5355 50  0000 L CNN
-F 2 "Package_SO:SOIC-14_3.9x8.7mm_P1.27mm" H 6600 5400 50  0001 C CNN
-F 3 "https://www.ti.com/lit/ds/slos351e/slos351e.pdf" H 6650 5600 50  0001 C CNN
-	5    6600 5400
-	1    0    0    -1
-$EndComp
 $Comp
 L Device:R_US R7
@@
 L Device:D_Zener D4
 U 1 1 615916B8
-P 7800 4800
-F 0 "D4" V 7750 4500 50  0000 L CNN
-F 1 "MMSZ5238B" V 7850 4250 50  0000 L CNN
-F 2 "Diode_SMD:D_SOD-123" H 7800 4800 50  0001 C CNN
-F 3 "https://www.diodes.com/assets/Datasheets/ds18010.pdf" H 7800 4800 50  0001 C CNN
-	1    7800 4800
+P 7100 4650
+F 0 "D4" V 7050 4350 50  0000 L CNN
+F 1 "MMSZ5238B" V 7150 4100 50  0000 L CNN
+F 2 "Diode_SMD:D_SOD-123" H 7100 4650 50  0001 C CNN
+F 3 "https://www.diodes.com/assets/Datasheets/ds18010.pdf" H 7100 4650 50  0001 C CNN
+	1    7100 4650
 	0    1    1    0
 $EndComp
@@
 L Device:LED D3
 U 1 1 61592B68
-P 7800 5100
-F 0 "D3" V 7839 4982 50  0000 R CNN
-F 1 "LED" V 7748 4982 50  0000 R CNN
-F 2 "LED_THT:LED_D3.0mm" H 7800 5100 50  0001 C CNN
-F 3 "~" H 7800 5100 50  0001 C CNN
-	1    7800 5100
+P 7100 4950
+F 0 "D3" V 7139 4832 50  0000 R CNN
+F 1 "LED" V 7048 4832 50  0000 R CNN
+F 2 "LED_THT:LED_D3.0mm" H 7100 4950 50  0001 C CNN
+F 3 "~" H 7100 4950 50  0001 C CNN
+	1    7100 4950
 	0    1    -1   0
 $EndComp
@@
 L Device:R_US R8
 U 1 1 61598D36
-P 7800 4500
-F 0 "R8" H 7733 4454 50  0000 R CNN
-F 1 "470" H 7733 4545 50  0000 R CNN
-F 2 "Resistor_SMD:R_0603_1608Metric_Pad0.98x0.95mm_HandSolder" V 7840 4490 50  0001 C CNN
-F 3 "~" H 7800 4500 50  0001 C CNN
-	1    7800 4500
+P 7100 4350
+F 0 "R8" H 7033 4304 50  0000 R CNN
+F 1 "470" H 7033 4395 50  0000 R CNN
+F 2 "Resistor_SMD:R_0603_1608Metric_Pad0.98x0.95mm_HandSolder" V 7140 4340 50  0001 C CNN
+F 3 "~" H 7100 4350 50  0001 C CNN
+	1    7100 4350
 	1    0    0    1
 $EndComp
-Wire Wire Line
-	7800 5250 7950 5250
 Connection ~ 7950 5250
 Wire Wire Line
@@
 U 2 1 615D3926
 P 6700 4000
-F 0 "Q9" V 6400 3850 50  0000 C CNN
-F 1 "SQ3989EV" V 6550 3750 50  0000 C CNN
+F 0 "Q9" H 6850 4400 50  0000 C CNN
+F 1 "SQ3989EV" H 6850 4300 50  0000 C CNN
 F 2 "Package_TO_SOT_SMD:TSOT-23-6_HandSoldering" H 6750 4000 50  0001 C CNN
 F 3 "https://www.vishay.com/docs/75059/sq3989ev.pdf" H 6750 4000 50  0001 C CNN
@@
 U 1 1 615D70CD
 P 6100 4000
-F 0 "Q9" V 5800 3850 50  0000 C CNN
-F 1 "SQ3989EV" V 5950 3750 50  0000 C CNN
+F 0 "Q9" H 6100 4400 50  0000 C CNN
+F 1 "SQ3989EV" H 6100 4300 50  0000 C CNN
 F 2 "Package_TO_SOT_SMD:TSOT-23-6_HandSoldering" H 6150 4000 50  0001 C CNN
 F 3 "https://www.vishay.com/docs/75059/sq3989ev.pdf" H 6150 4000 50  0001 C CNN
@@
 $EndComp
 Connection ~ 6800 4200
-Wire Wire Line
-	6800 4200 7100 4200
 Connection ~ 6800 3800
 Wire Wire Line
@@
 U 1 1 615DD480
 P 4500 5050
-F 0 "Q7" V 4850 5050 50  0000 C CNN
-F 1 "SQ3989EV" V 4700 5050 50  0000 C CNN
+F 0 "Q7" V 4650 5650 50  0000 C CNN
+F 1 "SQ3989EV" V 4550 5650 50  0000 C CNN
 F 2 "Package_TO_SOT_SMD:TSOT-23-6_HandSoldering" H 4550 5050 50  0001 C CNN
 F 3 "https://www.vishay.com/docs/75059/sq3989ev.pdf" H 4550 5050 50  0001 C CNN
@@
 U 2 1 615DDFBC
 P 4500 5500
-F 0 "Q7" H 4350 5750 50  0000 C CNN
-F 1 "SQ3989EV" H 4350 5650 50  0000 C CNN
+F 0 "Q7" V 4650 6100 50  0000 C CNN
+F 1 "SQ3989EV" V 4550 6100 50  0000 C CNN
 F 2 "Package_TO_SOT_SMD:TSOT-23-6_HandSoldering" H 4550 5500 50  0001 C CNN
 F 3 "https://www.vishay.com/docs/75059/sq3989ev.pdf" H 4550 5500 50  0001 C CNN
@@
 U 1 1 615DE779
 P 4500 4600
-F 0 "Q8" V 4500 4300 50  0000 C CNN
-F 1 "SQ3989EV" V 4400 4300 50  0000 C CNN
+F 0 "Q8" V 4750 4900 50  0000 C CNN
+F 1 "SQ3989EV" V 4650 4900 50  0000 C CNN
 F 2 "Package_TO_SOT_SMD:TSOT-23-6_HandSoldering" H 4550 4600 50  0001 C CNN
 F 3 "https://www.vishay.com/docs/75059/sq3989ev.pdf" H 4550 4600 50  0001 C CNN
@@
 U 2 1 615DF2CF
 P 2650 3000
-F 0 "Q1" V 2650 3300 50  0000 C CNN
-F 1 "SQ3989EV" V 2550 3300 50  0000 C CNN
+F 0 "Q1" V 3000 3000 50  0000 C CNN
+F 1 "SQ3989EV" V 2900 3000 50  0000 C CNN
 F 2 "Package_TO_SOT_SMD:TSOT-23-6_HandSoldering" H 2700 3000 50  0001 C CNN
 F 3 "https://www.vishay.com/docs/75059/sq3989ev.pdf" H 2700 3000 50  0001 C CNN
@@
 Wire Wire Line
 	2500 4300 2800 4300
-Wire Wire Line
-	7600 4350 7800 4350
-Connection ~ 7800 4350
-Wire Wire Line
-	7800 4350 8050 4350
 Text Label 3900 4300 0    50   ~ 0
 Vin
@@
 	8350 2800 8350 2950
 $Comp
-L Switch:SW_SPDT SW?
+L Switch:SW_SPDT SW4
 U 1 1 6193CCD8
 P 9550 4250
-F 0 "SW?" V 9596 4062 50  0000 R CNN
+F 0 "SW4" V 9596 4062 50  0000 R CNN
 F 1 "SW_SPDT" V 9505 4062 50  0000 R CNN
 F 2 "" H 9550 4250 50  0001 C CNN
@@
 Wire Wire Line
 	9650 4050 9900 4050
+Wire Wire Line
+	7600 4350 8050 4350
+Wire Wire Line
+	6800 4200 7100 4200
+Wire Wire Line
+	7100 5250 7100 5100
+Wire Wire Line
+	7100 5250 7950 5250
+$Comp
+L Amplifier_Operational:TLC274 U1
+U 1 1 6175147A
+P 5700 4200
+F 0 "U1" H 5200 4300 50  0000 C CNN
+F 1 "TLC274" H 5250 4200 50  0000 C CNN
+F 2 "Package_SO:SOIC-14_3.9x8.7mm_P1.27mm" H 5650 4300 50  0001 C CNN
+F 3 "https://www.ti.com/lit/ds/slos351e/slos351e.pdf" H 5750 4400 50  0001 C CNN
+	1    5700 4200
+	1    0    0    -1
+$EndComp
+$Comp
+L Amplifier_Operational:TLC274 U1
+U 5 1 61756E65
+P 6600 5400
+F 0 "U1" H 6558 5446 50  0000 L CNN
+F 1 "TLC274" H 6558 5355 50  0000 L CNN
+F 2 "Package_SO:SOIC-14_3.9x8.7mm_P1.27mm" H 6550 5500 50  0001 C CNN
+F 3 "https://www.ti.com/lit/ds/slos351e/slos351e.pdf" H 6650 5600 50  0001 C CNN
+	5    6600 5400
+	1    0    0    -1
+$EndComp
 $EndSCHEMATC
